File: templates/apex-template-2026/apex-template-2026.kicad_sch (KiCad schematic)
At the start: 0 parts

Commit message: First library additions
Parts:
- added H1, H2, H3, H4: M3 MH w/Pad, APEX_FOOTPRINTS:MH_M3-Pad, symbol APEX_Symbols:M3_Pad
- added U1: ADXL375, APEX_FOOTPRINTS:ADXL375_LGA_CC-14-1_ADI, symbol APEX_Symbols:ADXL375
- added U2: MMC5983MA, APEX_FOOTPRINTS:MMC5983MA_MEM, symbol APEX_Symbols:MMC5983MA
- added U3: ICM-45686, APEX_FOOTPRINTS:ICM-45686_LGA14L_TDK, symbol APEX_Symbols:ICM-45686
- added U4: BMP581, APEX_FOOTPRINTS:BMP581_QFN10_BOS, symbol APEX_Symbols:BMP581
Connections:
- new net GND: H1.1 (Pad), H2.1 (Pad), H3.1 (Pad), H4.1 (Pad)
