File: templates/apex-template-2026/apex-template-2026.kicad_sch (KiCad schematic)
At the start: 8 parts, among them U1 ADXL375, U2 MMC5983MA, U3 ICM-45686, U4 BMP581

Commit message: Project split
Parts:
- removed U1: ADXL375, APEX_FOOTPRINTS:ADXL375_LGA_CC-14-1_ADI, symbol APEX_Symbols:ADXL375
- removed U2: MMC5983MA, APEX_FOOTPRINTS:MMC5983MA_MEM, symbol APEX_Symbols:MMC5983MA
- removed U3: ICM-45686, APEX_FOOTPRINTS:ICM-45686_LGA14L_TDK, symbol APEX_Symbols:ICM-45686
- removed U4: BMP581, APEX_FOOTPRINTS:BMP581_QFN10_BOS, symbol APEX_Symbols:BMP581
