File: templates/apex-template-2026/apex-template-2026.kicad_pcb (KiCad board)
At the start: 4 copper layers, 50 x 50 mm, 8 parts, among them U1 ADXL375, U2 MMC5983MA, U3 ICM-45686, U4 BMP581

Commit message: Added MAX-M10S-00B footprint
Parts:
- added REF**: XCVR_MAX-M10S-00B, APEX_FOOTPRINTS:MAX-M10S-00B_XCVR, F.Cu at (87.0, 86.5)
