File: templates/apex-template-2026/apex-template-2026.kicad_pcb (KiCad board)
At the start: 2 copper layers, 50 x 50 mm, 0 parts

Commit message: First template version
Routing:
- net (no net): vias 0 -> 1
Other:
- copper layers 2 -> 4
Changed lines of the file:
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@@
 	(generator_version "10.0")
 	(general
-		(thickness 1.6)
+		(thickness 1.6062)
 		(legacy_teardrops no)
 	)
@@
 	(layers
 		(0 "F.Cu" signal)
+		(4 "In1.Cu" power)
+		(6 "In2.Cu" power)
 		(2 "B.Cu" signal)
 		(9 "F.Adhes" user "F.Adhesive")
@@
 	)
 	(setup
+		(stackup
+			(layer "F.SilkS"
+				(type "Top Silk Screen")
+				(color "White")
+			)
+			(layer "F.Paste"
+				(type "Top Solder Paste")
+			)
+			(layer "F.Mask"
+				(type "Top Solder Mask")
+				(color "Green")
+				(thickness 0.01)
+			)
+			(layer "F.Cu"
+				(type "copper")
+				(thickness 0.035)
+			)
+			(layer "dielectric 1"
+				(type "prepreg")
+				(color "FR4 natural")
+				(thickness 0.2104)
+				(material "FR4")
+				(epsilon_r 4.4)
+				(loss_tangent 0.02)
+			)
+			(layer "In1.Cu"
+				(type "copper")
+				(thickness 0.0152)
+			)
+			(layer "dielectric 2"
+				(type "core")
+				(color "FR4 natural")
+				(thickness 1.065)
+				(material "FR4")
+				(epsilon_r 4.6)
+				(loss_tangent 0.02)
+			)
+			(layer "In2.Cu"
+				(type "copper")
+				(thickness 0.0152)
+			)
+			(layer "dielectric 3"
+				(type "prepreg")
+				(color "FR4 natural")
+				(thickness 0.2104)
+				(material "FR4")
+				(epsilon_r 4.4)
+				(loss_tangent 0.02)
+			)
+			(layer "B.Cu"
+				(type "copper")
+				(thickness 0.035)
+			)
+			(layer "B.Mask"
+				(type "Bottom Solder Mask")
+				(color "Green")
+				(thickness 0.01)
+			)
+			(layer "B.Paste"
+				(type "Bottom Solder Paste")
+			)
+			(layer "B.SilkS"
+				(type "Bottom Silk Screen")
+				(color "White")
+			)
+			(copper_finish "HAL SnPb")
+			(dielectric_constraints no)
+		)
 		(pad_to_mask_clearance 0)
 		(allow_soldermask_bridges_in_footprints no)
@@
 		(capping no)
 		(filling no)
+		(zone_defaults)
 		(pcbplotparams
 			(layerselection 0x00000000_00000000_55555555_5755f5ff)
@@
 	)
 	(gr_rect
-		(start 109.5 68)
-		(end 159.5 118)
+		(start 76 76)
+		(end 124 124)
+		(radius 4.5)
+		(stroke
+			(width 0.3)
+			(type solid)
+		)
+		(fill no)
+		(layer "F.SilkS")
+	)
+	(gr_rect
+		(start 75 75)
+		(end 125 125)
 		(radius 5)
 		(stroke
@@
 		(layer "Edge.Cuts")
 	)
+	(via
+		(at 80.25 80.25)
+		(size 3.6)
+		(drill 3)
+		(layers "F.Cu" "B.Cu")
+		(net "")
+	)
 	(embedded_fonts no)

Commit message: First library additions
Parts:
- added H1: M3 MH w/Pad, APEX_FOOTPRINTS:MH_M3-Pad, F.Cu at (3.02, 3.02)
- added H2: M3 MH w/Pad, APEX_FOOTPRINTS:MH_M3-Pad, F.Cu at (3.02, 10.1)
- added H3: M3 MH w/Pad, APEX_FOOTPRINTS:MH_M3-Pad, F.Cu at (3.02, 17.1)
- added H4: M3 MH w/Pad, APEX_FOOTPRINTS:MH_M3-Pad, F.Cu at (3.02, 24.2)
- added U1: ADXL375, APEX_FOOTPRINTS:ADXL375_LGA_CC-14-1_ADI, F.Cu at (101.8, 100.1)
- added U2: MMC5983MA, APEX_FOOTPRINTS:MMC5983MA_MEM, F.Cu at (93.7, 98.2)
- added U3: ICM-45686, APEX_FOOTPRINTS:ICM-45686_LGA14L_TDK, F.Cu at (100.1, 88.3)
- added U4: BMP581, APEX_FOOTPRINTS:BMP581_QFN10_BOS, F.Cu at (107.0, 91.5)
Routing:
- net (no net): vias 1 -> 0

Commit message: Project split
Parts:
- removed H1, H2, H3, H4: M3 MH w/Pad, APEX_FOOTPRINTS:MH_M3-Pad
- removed U1: ADXL375, APEX_FOOTPRINTS:ADXL375_LGA_CC-14-1_ADI
- removed U2: MMC5983MA, APEX_FOOTPRINTS:MMC5983MA_MEM
- removed U3: ICM-45686, APEX_FOOTPRINTS:ICM-45686_LGA14L_TDK
- removed U4: BMP581, APEX_FOOTPRINTS:BMP581_QFN10_BOS
Other:
- board outline removed
