File: boards/apex_control/sensors.kicad_sch (KiCad schematic)
At the start: 0 parts

Commit message: Logan done fo now
Parts:
- added U1: ADXL375, APEX_FOOTPRINTS:ADXL375_LGA_CC-14-1_ADI, symbol APEX_Symbols:ADXL375
- added U2: MMC5983MA, APEX_FOOTPRINTS:MMC5983MA_MEM, symbol APEX_Symbols:MMC5983MA
- added U3: ICM-45686, APEX_FOOTPRINTS:ICM-45686_LGA14L_TDK, symbol APEX_Symbols:ICM-45686
- added U4: BMP581, APEX_FOOTPRINTS:BMP581_QFN10_BOS, symbol APEX_Symbols:BMP581
- added U5: RTMC-G2-4IQ48, APEX_FOOTPRINTS:RTMC-G2-4IQ48_LQFP-48_ThetaMachines, symbol APEX_Symbols:RTMC-G2-4IQ48
Connections:
- new net GND: U5.14 (GND), U5.19 (GND), U5.27 (GND), U5.35 (GND), U5.45 (GND), U5.6 (GND)
- new net VDD: U5.15 (VDD), U5.20 (VDD), U5.28 (VDD), U5.36 (VDD), U5.46 (VDD), U5.7 (VDD)
