File: boards/apex_control/apex-control-2026.kicad_pcb (KiCad board)
At the start: 4 copper layers, 50 x 100 mm, 4 parts

Commit message: Logan done fo now
Parts:
- added J1: UJ20-C-H-G-SMT-5-P16, APEX_FOOTPRINTS:UJ20-C-H-G-SMT-5-P16_SameSky, F.Cu at (79.0, 64.5)
- added U1: ADXL375, APEX_FOOTPRINTS:ADXL375_LGA_CC-14-1_ADI, F.Cu at (112.4, 127.8)
- added U10: MKL26Z128VFM4, APEX_FOOTPRINTS:MKL26Z128VFM4_QFN32_NXP, F.Cu at (96.3, 69.8)
- added U11: W25Q64JW, APEX_FOOTPRINTS:W25Q64JW_USON8_Winbond, F.Cu at (104.2, 70.7)
- added U12: MAYA-W166-00B, APEX_FOOTPRINTS:MAYA-W166_LGA86_u-blox, F.Cu at (117.7, 84.0)
- added U2: MMC5983MA, APEX_FOOTPRINTS:MMC5983MA_MEM, F.Cu at (112.4, 133.6)
- added U3: ICM-45686, APEX_FOOTPRINTS:ICM-45686_LGA14L_TDK, F.Cu at (100.3, 138.1)
- added U4: BMP581, APEX_FOOTPRINTS:BMP581_QFN10_BOS, F.Cu at (104.8, 138.1)
- added U5: RTMC-G2-4IQ48, APEX_FOOTPRINTS:RTMC-G2-4IQ48_LQFP-48_ThetaMachines, F.Cu at (102.2, 125.0)
- added U6: MIMXRT1171DVMAB, APEX_FOOTPRINTS:MIMXRT1171DVMAB_BGA, F.Cu at (100.8, 84.1)
- added U7: TPS62086, APEX_FOOTPRINTS:TPS62086_RLT0007A_TI, F.Cu at (110.1, 67.5)
- added U8: TPS62825, APEX_FOOTPRINTS:TPS62825_DMQ0006A_TI, F.Cu at (113.5, 70.8)
- added U9: LM66200, APEX_FOOTPRINTS:LM66200_DRL0008A_TI, F.Cu at (109.9, 71.2)
- added Y1: Crystal_GND24, APEX_FOOTPRINTS:XTAL_3225, F.Cu at (90.8, 90.0)

Commit message: More placement
Parts:
- added REF**: SAMTEC_EHF-120-01-L-D, APEX_FOOTPRINTS:SAMTEC_EHF-120-01-L-D, F.Cu at (137.8, 127.2)
- added REF**: SAMTEC_EHF-120-01-L-D, APEX_FOOTPRINTS:SAMTEC_EHF-120-01-L-D, F.Cu at (120.0, 120.0)
- added REF**: SAMTEC_EHF-120-01-L-D, APEX_FOOTPRINTS:SAMTEC_EHF-120-01-L-D, F.Cu at (80.8, 120.8)
- added REF**: SAMTEC_EHF-120-01-L-D, APEX_FOOTPRINTS:SAMTEC_EHF-120-01-L-D, F.Cu at (64.2, 128.0)
- moved J1 23.5 mm to (100.0, 53.9), turned to 180 degrees
- moved U2 23.4 mm to (97.5, 115.5)
- moved U1 13.1 mm to (108.5, 115.2)
- moved U4 6.58 mm to (109.0, 133.0)
- moved U3 5.65 mm to (97.5, 133.2)
Other:
- board size 50 x 100 mm -> 147.5 x 100.5 mm

Commit message: Worked on stuff
Parts:
- removed REF** (x4): SAMTEC_EHF-120-01-L-D, APEX_FOOTPRINTS:SAMTEC_EHF-120-01-L-D
- moved J1 23.5 mm to (79.0, 64.5), turned to -90 degrees
- moved U2 23.4 mm to (112.4, 133.6)
- moved U1 13.1 mm to (112.4, 127.8)
- moved U4 6.58 mm to (104.8, 138.1)
- moved U3 5.65 mm to (100.3, 138.1)
Other:
- board size 147.5 x 100.5 mm -> 50 x 100 mm
