File: boards/apex_control/user-IO.kicad_sch (KiCad schematic)
At the start: 0 parts

Commit message: Logan done fo now
Parts:
- added U12: MAYA-W166-00B, APEX_FOOTPRINTS:MAYA-W166_LGA86_u-blox, symbol APEX_Symbols:MAYA-W166-00B
- added U6: MIMXRT1171DVMAB, APEX_FOOTPRINTS:MIMXRT1171DVMAB_BGA, symbol APEX_Symbols:MIMXRT1171DVMAB
Connections:
- new net: U12.J7 (BT_RESET), U6.A16 (GPIO_SD_B1_05)
- new net: U12.J3 (PDn), U6.A3 (GPIO_EMC_B1_09)
- new net: U12.J8 (WLAN_DEV_WAKE), U6.A4 (GPIO_DISP_B2_15)
- new net: U12.H8 (UART_CTSn), U6.A5 (GPIO_DISP_B2_13)
- new net: U12.G9 (UART_SOUT), U6.A6 (GPIO_DISP_B2_11)
- new net: U12.J9 (BT_DEV_WAKE), U6.A7 (GPIO_DISP_B2_14)
- new net: U12.E7 (BT_WAKE_HOST), U6.B16 (GPIO_SD_B1_00)
- new net: U12.F7 (WLAN_WAKE_HOST), U6.B17 (GPIO_SD_B1_03)
- new net: U12.H9 (UART_RTSn), U6.B6 (GPIO_DISP_B2_12)
- new net: U12.H7 (WLAN_RESET), U6.C15 (GPIO_SD_B1_02)
- new net: U12.G8 (UART_SIN), U6.D9 (GPIO_DISP_B2_10)
- new net: U12.B4 (SD_CMD), U6.E14 (GPIO_SD_B2_05)
- new net: U12.B3 (SD_DAT[0]), U6.E15 (GPIO_SD_B2_03)
- new net: U12.A4 (SD_CLK), U6.F14 (GPIO_SD_B2_04)
- new net: U12.A3 (SD_DAT[1]), U6.H13 (GPIO_SD_B2_02)
- new net: U12.B5 (SD_DAT[2]), U6.J14 (GPIO_SD_B2_01)
- new net: U12.A5 (SD_DAT[3]), U6.J15 (GPIO_SD_B2_00)
- new net: U12.A1 (GND), U12.A9 (GND), U12.B2 (GND), U12.B8 (GND), U12.E4 (GND), U12.E5 (GND), U12.F4 (GND), U12.F5 (GND), U12.H4 (GND), U12.H5 (GND), U12.K2 (GND), U12.K3 (GND), U12.K4 (GND), U12.K6 (GND), U12.K7 (GND), U12.K8 (GND), U12.L1 (GND), U12.L9 (GND), U12.M1 (GND), U12.M2 (GND), U12.M8 (GND), U12.M9 (GND)
- new net: U12.A7 (3V3), U12.B7 (3V3)

Commit message: Worked on stuff
Parts:
- added R22: R, symbol APEX_Symbols:R
Connections:
- net GND: now reaches U12.A1 (GND), U12.A9 (GND), U12.B2 (GND), U12.B8 (GND), U12.E4 (GND), U12.E5 (GND), U12.F4 (GND), U12.F5 (GND), U12.H4 (GND), U12.H5 (GND), U12.K2 (GND), U12.K3 (GND), U12.K4 (GND), U12.K6 (GND), U12.K7 (GND), U12.K8 (GND), U12.L1 (GND), U12.L9 (GND), U12.M1 (GND), U12.M2 (GND), U12.M8 (GND), U12.M9 (GND)
- net GND: now also R22.2
- net +1V8: now reaches U12.A2 (1V8)
- net +1V8: now also U12.A6 (VIO_SD), U12.A8 (VIO)
- net +3V3_1: now reaches U12.A7 (3V3), U12.B7 (3V3)
- net at U12.D3 (CONFIG[0]): now also R22.1
- no-connect marks 0 -> 1
