File: boards/apex_telemetry/apex-telemetry-2026.kicad_pcb (KiCad board)
At the start: 4 copper layers, 0 parts

Commit message: Added board outline and placed holes
Parts:
- added H1: M3 MH w/Pad, APEX_FOOTPRINTS:MH_M3-Pad, F.Cu at (82.5, 82.5)
- added H2: M3 MH w/Pad, APEX_FOOTPRINTS:MH_M3-Pad, F.Cu at (117.5, 82.5)
- added H3: M3 MH w/Pad, APEX_FOOTPRINTS:MH_M3-Pad, F.Cu at (82.5, 117.5)
- added H4: M3 MH w/Pad, APEX_FOOTPRINTS:MH_M3-Pad, F.Cu at (117.5, 117.5)
Other:
- board outline added: 45 x 45 mm
